Commit message: Added change to incorporate plate frame.

File: urdf/med.urdf (robot description, URDF)
Before this commit: robot iiwa, 11 links, 10 joints
Joints:
- joint iiwa_joint_ee: origin xyz=0 0 0.045 rpy=3.141592653589793 3.141592653589793 3.141592653589793 -> xyz=0 0 0.035 rpy=3.141592653589793 3.141592653589793 3.141592653589793
- joint tool0_joint: origin xyz=0 0 0.045 rpy=0 -1.570796326794897 0 -> xyz=0 0 0.035 rpy=0 -1.570796326794897 0
