Commit message: Fixed urdf bug. Lets start taking out hacks.

File: urdf/med_gamma.urdf (robot description, URDF)
Before this commit: robot iiwa, 11 links, 10 joints
Joints:
- joint iiwa_joint_ee: origin xyz=0 0 0.085 rpy=3.141592653589793 3.141592653589793 3.141592653589793 -> xyz=0 0 0.0775 rpy=3.141592653589793 3.141592653589793 3.141592653589793
- joint tool0_joint: origin xyz=0 0 0.085 rpy=0 -1.570796326794897 0 -> xyz=0 0 0.0775 rpy=0 -1.570796326794897 0

File: urdf/med_gamma_shorter.urdf (robot description, URDF)
Before this commit: robot iiwa, 11 links, 10 joints
Joints:
- joint iiwa_joint_ee: origin xyz=0 0 0.08 rpy=3.141592653589793 3.141592653589793 3.141592653589793 -> xyz=0 0 0.0725 rpy=3.141592653589793 3.141592653589793 3.141592653589793
- joint tool0_joint: origin xyz=0 0 0.08 rpy=0 -1.570796326794897 0 -> xyz=0 0 0.0725 rpy=0 -1.570796326794897 0
