Commit message: Added all changes for algorithm. Currently algorithm is causing pandas to collide.

File: urdf/franka_description/panda_arm.urdf (robot description, URDF)
Before this commit: robot panda, 9 links, 8 joints
Links:
- link panda_link0: geometry visual mesh filename=package://drake_models/franka_description/meshes/visual/lin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
- link panda_link1: geometry visual mesh filename=package://drake_models/franka_description/meshes/visual/lin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
- link panda_link2: geometry visual mesh filename=package://drake_models/franka_description/meshes/visual/lin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
- link panda_link3: geometry visual mesh filename=package://drake_models/franka_description/meshes/visual/lin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
- link panda_link4: geometry visual mesh filename=package://drake_models/franka_description/meshes/visual/lin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
- link panda_link5: geometry visual mesh filename=package://drake_models/franka_description/meshes/visual/lin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
- link panda_link6: geometry visual mesh filename=package://drake_models/franka_description/meshes/visual/lin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
- link panda_link7: geometry visual mesh filename=package://drake_models/franka_description/meshes/visual/lin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
- link panda_link8: geometry 
